File: E104-BT11/E104-BT11G-PCB.brd (EAGLE design)
At the start: 20.1 x 35.3 mm, 3 parts

Commit message: Add files via upload
Parts:
- added BOOT, RST: SKRKAEE010, button3:SKRK
- added C1: (no value), Capacitor:CAPM3528X210
- added J3: (no value), SparkFun-Connectors:1X04_NO_SILK
- added LINK: (no value), adafruit:CHIP-LED0603
- added R1: 2.2k, SparkFun-Resistors:0603
- added R2: 150R, SparkFun-Resistors:0603
Connections:
- new net N$1: LINK.C, R1.2
- new net N$2: BOOT.1, R2.2
- net GND: now also C1.2, J3.1, R2.1, RST.1
- net NETL: now also R1.1
- net PA00: now also BOOT.2
- net RST: now also RST.2
- net RXD: now also J3.3
- net TXD: now also J3.4
- net VCC: now also C1.1, J3.2, LINK.A
Routing:
- net RST: track 2.79 -> 31.4 mm, vias 0 -> 2
- net VCC: track 39.4 -> 62.5 mm, vias 1 -> 2
- net RXD: track 9.23 -> 29.9 mm
- net PA00: track 7.44 -> 26.0 mm
- net TXD: track 10.9 -> 26.7 mm
- net NETL: track 24.7 -> 29.4 mm
- net N$2: track 0.00 -> 3.85 mm
- net N$1: track 0.00 -> 2.30 mm
- net SWD: track 16.5 -> 18.6 mm
Other:
- board text added: "BOOT"
- board text added: "C1"
- board text added: "NETL"
- board text added: "RST"
- board text added: "TCK/SWC"
- board text added: "TDI/PA04"
- board text added: "TDO/PA03"
- board text added: "TMS/SWD"
- board text removed: "PA03"
- board text removed: "PA04"
- board text removed: "SWC"
- board text removed: "SWD"

Commit message: Add files via upload
Parts:
- C1: value (none) -> 220u
Connections:
- net NC_3: now also J1.7; no longer J1.5
- net PA03: now also J1.6; no longer J1.10
- net PA04: now also J1.5; no longer J1.7
- net PA05: now also J1.10; no longer J1.6
Routing:
- net PA03: track 8.24 -> 20.0 mm
- net PA05: track 13.9 -> 2.59 mm, vias 1 -> 0
- net PA04: track 12.3 -> 19.9 mm, vias 1 -> 2
- net PA00: track 26.0 -> 32.4 mm
- net NC_3: track 18.9 -> 14.6 mm
- net VCC: track 62.5 -> 63.2 mm
- net NC_1: track 9.51 -> 10.0 mm
