File: E104-BT11/E104-BT11G-PCB.sch (EAGLE design)
At the start: 3 parts

Commit message: Add files via upload
Parts:
- added BOOT, RST: SKRKAEE010, button3:SKRKAEE010
- added C1: (no value), Capacitor:C_TANTALUM-1411(3528-METRIC)
- added J3: (no value), SparkFun-Connectors:CONN_041X04_NO_SILK
- added LINK: (no value), adafruit:LEDCHIP-LED0603
- added R1: 2.2k, SparkFun-Resistors:2.2KOHM-0603-1/10W-1%
- added R2: 150R, SparkFun-Resistors:2.2KOHM-0603-1/10W-1%
Connections:
- new net N$1: LINK.C, R1.2
- new net N$2: BOOT.1, R2.2
- net GND: now also C1.2, J3.1, R2.1, RST.1
- net NETL: now also R1.1
- net PA00: now also BOOT.2
- net RST: now also RST.2
- net RXD: now also J3.3
- net TXD: now also J3.4
- net VCC: now also C1.1, J3.2, LINK.A
Other:
- moved on the sheet: J1, J2

Commit message: Add files via upload
Parts:
- C1: value (none) -> 220u
Connections:
- net NC_3: now also J1.7; no longer J1.5
- net PA03: now also J1.6; no longer J1.10
- net PA04: now also J1.5; no longer J1.7
- net PA05: now also J1.10; no longer J1.6
Changed lines of the file:
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@@
 <part name="LINK" library="adafruit" library_urn="urn:adsk.eagle:library:420" deviceset="LED" device="CHIP-LED0603" package3d_urn="urn:adsk.eagle:package:6240556/1"/>
 <part name="R1" library="SparkFun-Resistors" library_urn="urn:adsk.eagle:library:532" deviceset="2.2KOHM" device="-0603-1/10W-1%" package3d_urn="urn:adsk.eagle:package:39650/1" value="2.2k"/>
-<part name="C1" library="Capacitor" library_urn="urn:adsk.eagle:library:16290819" deviceset="C" device="TANTALUM-1411(3528-METRIC)" package3d_urn="urn:adsk.eagle:package:16290902/2" technology="_"/>
+<part name="C1" library="Capacitor" library_urn="urn:adsk.eagle:library:16290819" deviceset="C" device="TANTALUM-1411(3528-METRIC)" package3d_urn="urn:adsk.eagle:package:16290902/2" technology="_" value="220u"/>
 <part name="GND1" library="supply1" library_urn="urn:adsk.eagle:library:371" deviceset="GND" device=""/>
 <part name="BOOT" library="button3" deviceset="SKRKAEE010" device=""/>
@@
 </instance>
 <instance part="C1" gate="G$1" x="116.84" y="38.1" smashed="yes" rot="R90">
-<attribute name="NAME" x="114.3" y="40.64" size="1.778" layer="95"/>
-<attribute name="VALUE" x="116.84" y="40.64" size="1.778" layer="96" rot="R90"/>
+<attribute name="NAME" x="116.84" y="40.64" size="1.778" layer="95"/>
+<attribute name="VALUE" x="121.92" y="35.56" size="1.778" layer="96" rot="R180"/>
 </instance>
 <instance part="GND1" gate="1" x="124.46" y="30.48" smashed="yes">
@@
 <net name="PA03" class="0">
 <segment>
+<pinref part="U$1" gate="G$1" pin="PA03"/>
+<wire x1="60.96" y1="45.72" x2="50.8" y2="45.72" width="0.1524" layer="91"/>
+<label x="50.8" y="45.72" size="1.778" layer="95"/>
+</segment>
+<segment>
+<pinref part="J1" gate="G$1" pin="6"/>
+<wire x1="12.7" y1="35.56" x2="20.32" y2="35.56" width="0.1524" layer="91"/>
+<label x="15.24" y="35.56" size="1.778" layer="95"/>
+</segment>
+</net>
+<net name="NC_1" class="0">
+<segment>
+<pinref part="J1" gate="G$1" pin="9"/>
+<wire x1="12.7" y1="43.18" x2="20.32" y2="43.18" width="0.1524" layer="91"/>
+<label x="15.24" y="43.18" size="1.778" layer="95"/>
+</segment>
+<segment>
+<pinref part="U$1" gate="G$1" pin="NC@1"/>
+<wire x1="60.96" y1="43.18" x2="50.8" y2="43.18" width="0.1524" layer="91"/>
+<label x="50.8" y="43.18" size="1.778" layer="95"/>
+</segment>
+</net>
+<net name="NC_2" class="0">
+<segment>
+<pinref part="J1" gate="G$1" pin="8"/>
+<wire x1="12.7" y1="40.64" x2="20.32" y2="40.64" width="0.1524" layer="91"/>
+<label x="15.24" y="40.64" size="1.778" layer="95"/>
+</segment>
+<segment>
+<pinref part="U$1" gate="G$1" pin="NC@2"/>
+<wire x1="60.96" y1="40.64" x2="50.8" y2="40.64" width="0.1524" layer="91"/>
+<label x="50.8" y="40.64" size="1.778" layer="95"/>
+</segment>
+</net>
+<net name="PA04" class="0">
+<segment>
+<pinref part="U$1" gate="G$1" pin="PA04"/>
+<wire x1="60.96" y1="38.1" x2="50.8" y2="38.1" width="0.1524" layer="91"/>
+<label x="50.8" y="38.1" size="1.778" layer="95"/>
+</segment>
+<segment>
+<pinref part="J1" gate="G$1" pin="5"/>
+<wire x1="12.7" y1="33.02" x2="20.32" y2="33.02" width="0.1524" layer="91"/>
+<label x="15.24" y="33.02" size="1.778" layer="95"/>
+</segment>
+</net>
+<net name="PA05" class="0">
+<segment>
+<pinref part="U$1" gate="G$1" pin="PA05"/>
+<wire x1="60.96" y1="35.56" x2="50.8" y2="35.56" width="0.1524" layer="91"/>
+<label x="50.8" y="35.56" size="1.778" layer="95"/>
+</segment>
+<segment>
 <pinref part="J1" gate="G$1" pin="10"/>
 <wire x1="12.7" y1="45.72" x2="20.32" y2="45.72" width="0.1524" layer="91"/>
 <label x="15.24" y="45.72" size="1.778" layer="95"/>
-</segment>
-<segment>
-<pinref part="U$1" gate="G$1" pin="PA03"/>
-<wire x1="60.96" y1="45.72" x2="50.8" y2="45.72" width="0.1524" layer="91"/>
-<label x="50.8" y="45.72" size="1.778" layer="95"/>
-</segment>
-</net>
-<net name="NC_1" class="0">
-<segment>
-<pinref part="J1" gate="G$1" pin="9"/>
-<wire x1="12.7" y1="43.18" x2="20.32" y2="43.18" width="0.1524" layer="91"/>
-<label x="15.24" y="43.18" size="1.778" layer="95"/>
-</segment>
-<segment>
-<pinref part="U$1" gate="G$1" pin="NC@1"/>
-<wire x1="60.96" y1="43.18" x2="50.8" y2="43.18" width="0.1524" layer="91"/>
-<label x="50.8" y="43.18" size="1.778" layer="95"/>
-</segment>
-</net>
-<net name="NC_2" class="0">
-<segment>
-<pinref part="J1" gate="G$1" pin="8"/>
-<wire x1="12.7" y1="40.64" x2="20.32" y2="40.64" width="0.1524" layer="91"/>
-<label x="15.24" y="40.64" size="1.778" layer="95"/>
-</segment>
-<segment>
-<pinref part="U$1" gate="G$1" pin="NC@2"/>
-<wire x1="60.96" y1="40.64" x2="50.8" y2="40.64" width="0.1524" layer="91"/>
-<label x="50.8" y="40.64" size="1.778" layer="95"/>
-</segment>
-</net>
-<net name="PA04" class="0">
-<segment>
-<pinref part="J1" gate="G$1" pin="7"/>
-<wire x1="12.7" y1="38.1" x2="20.32" y2="38.1" width="0.1524" layer="91"/>
-<label x="15.24" y="38.1" size="1.778" layer="95"/>
-</segment>
-<segment>
-<pinref part="U$1" gate="G$1" pin="PA04"/>
-<wire x1="60.96" y1="38.1" x2="50.8" y2="38.1" width="0.1524" layer="91"/>
-<label x="50.8" y="38.1" size="1.778" layer="95"/>
-</segment>
-</net>
-<net name="PA05" class="0">
-<segment>
-<pinref part="J1" gate="G$1" pin="6"/>
-<wire x1="12.7" y1="35.56" x2="20.32" y2="35.56" width="0.1524" layer="91"/>
-<label x="15.24" y="35.56" size="1.778" layer="95"/>
-</segment>
-<segment>
-<pinref part="U$1" gate="G$1" pin="PA05"/>
-<wire x1="60.96" y1="35.56" x2="50.8" y2="35.56" width="0.1524" layer="91"/>
-<label x="50.8" y="35.56" size="1.778" layer="95"/>
 </segment>
 </net>
@@
 </segment>
 <segment>
-<pinref part="J1" gate="G$1" pin="5"/>
-<wire x1="12.7" y1="33.02" x2="20.32" y2="33.02" width="0.1524" layer="91"/>
-<label x="15.24" y="33.02" size="1.778" layer="95"/>
-</segment>
-</net>
+<pinref part="J1" gate="G$1" pin="7"/>
+<wire x1="12.7" y1="38.1" x2="20.32" y2="38.1" width="0.1524" layer="91"/>
+<label x="15.24" y="38.1" size="1.778" layer="95"/>
+</segment>
+</net>
